File: Code/PCB/Hellfire.kicad_pcb (KiCad board)
At the start: 2 copper layers, 99.1 x 52.1 mm, 24 parts

Commit message: Hellfire+pcb update
Parts:
- moved NE1 4.12 mm to (107.8, 129.3), turned to -90 degrees
- moved R7 2.46 mm to (130.8, 133.3), turned to -90 degrees
- turned VR1 to -90 degrees
Routing:
- net (no net): track 80.7 -> 0.00 mm
- net Net-(NE1-Pad9): track 0.00 -> 34.4 mm
- net Net-(D5-K): track 144.6 -> 163.0 mm
- net Net-(NE1-Pad1): track 0.00 -> 16.1 mm
- net Net-(D5-A): track 46.3 -> 57.5 mm
- net Net-(BJ1-Pad3): track 45.2 -> 55.1 mm
- net Net-(R7-Pad1): track 15.6 -> 22.9 mm
- net Net-(BJ1-Pad2): track 63.9 -> 59.5 mm
- net Net-(NE1-Pad5): track 12.2 -> 13.6 mm
- net Net-(NE1-GND): track 131.0 -> 129.9 mm
